File: BGA2869 amplifier/BGA2869 amplifier.kicad_sch (KiCad schematic)
At the start: 19 parts, among them J1 Barrel_Jack_MountingPin, J2 USB_C_Receptacle_USB2.0_16P, J3 Conn_Coaxial, J4 Conn_Coaxial, U1 BGA2869

Commit message: MMBF5485 amp rev0
Parts:
- H4: footprint MountingHole:MountingHole_3.2mm_M3_DIN965_Pad_TopBottom -> MountingHole:MountingHole_3mm
Changed lines of the file:
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@@
 			)
 		)
-		(property "Footprint" "MountingHole:MountingHole_3.2mm_M3_DIN965_Pad_TopBottom"
+		(property "Footprint" "MountingHole:MountingHole_3mm"
 			(at 186.69 86.36 0)
 			(effects
